File: hardware/kbd-nes-v1/kbd-nes-v1.kicad_pcb (KiCad board)
At the start: 4 copper layers, 49.2 x 30.9 mm, 49 parts, among them J2 Conn_01x02, J3 USB_C_Receptacle_USB2.0_16P, J4 USB_C_Receptacle_USB2.0_16P, J5 Conn_01x05, J6 Conn_ARM_SWD_TagConnect_TC203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, Q1 2N7002, U2 W25Q128JVS, U3 RP2040, U4 AMS1117-3.3, U5 TPS2051BDR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

Commit message: final submitted CAD to JLC
Parts:
- U5: footprint Package_SO:SOIC-8_5.3x5.3mm_P1.27mm -> TI parts:D8
- moved U5 1.50 mm to (147.9, 77.4), turned to 0 degrees
Connections:
- U5 pad 1: /USB Keyboard Host/+5V_HOST -> GND
- U5 pad 2: GND -> /RP2040 Core/+5V_IN
- U5 pad 3: /RP2040 Core/FAULT_N -> /RP2040 Core/+5V_IN
- U5 pad 5: /RP2040 Core/+5V_IN -> /RP2040 Core/FAULT_N
- U5 pad 6: /RP2040 Core/+5V_IN -> /USB Keyboard Host/+5V_HOST
- U5 pad 7: /RP2040 Core/+5V_IN -> /USB Keyboard Host/+5V_HOST
- U5 pad 8: /RP2040 Core/+5V_IN -> /USB Keyboard Host/+5V_HOST
Routing:
- net /USB Keyboard Host/+5V_HOST: track 31.1 -> 43.8 mm
- net /RP2040 Core/HOST_VBUS_EN: track 29.1 -> 18.3 mm
- net /RP2040 Core/FAULT_N: track 56.1 -> 47.1 mm
- net /RP2040 Core/+5V_IN: track 46.6 -> 42.0 mm, vias 7 -> 5
