File: hardware/kbd-nes-v1/kbd-nes-v1.kicad_sch (KiCad schematic)
At the start: 0 parts

Commit message: final submitted CAD to JLC
Changed lines of the file:
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@@
 			)
 		)
-		(pin "FAULT_N" output
+		(pin "FAULT_N" input
 			(at 190.5 72.39 180)
 			(effects
