File: hardware/kbd-nes-v1/rp2040_core.kicad_sch (KiCad schematic)
At the start: 28 parts, among them J2 Conn_01x02, J6 Conn_ARM_SWD_TagConnect_TC203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, U2 W25Q128JVS, U3 RP2040, U4 AMS1117-3.3, Y1 ABM8-272-T3

Commit message: final submitted CAD to JLC
Parts:
- Y1: LCSC (none) -> C20625731
Changed lines of the file:
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@@
+			)
+		)
+		(property "LCSC" "C20625731 "
+			(at 63.5 154.94 90)
+			(hide yes)
+			(show_name no)
+			(do_not_autoplace no)
+			(effects
+				(font
+					(size 1.27 1.27)
+				)
 			)
 		)
