File: hardware/kbd-nes-v1/usb_keyboard_host.kicad_sch (KiCad schematic)
At the start: 7 parts, among them J4 USB_C_Receptacle_USB2.0_16P, U5 TPS2051BDR

Commit message: final submitted CAD to JLC
Parts:
- removed U5: TPS2051BDR, Package_SO:SOIC-8_5.3x5.3mm_P1.27mm, symbol Power_Management:TPS2051BDR
- added U5: TPS2051BDR, TI parts:D8, symbol Custom TI Power Switch:TPS2051BDR
Connections:
- net +5V_HOST: now also U5.6 (OUT), U5.7 (OUT), U5.8 (OUT)
- net +5V_IN: now also U5.2 (IN), U5.3 (IN)
- net FAULT_N: now also U5.5 (*OC)
- net HOST_VBUS_EN: now also U5.4 (*EN)
- net USB_HOST_GND: now also U5.1 (GND)
