File: hardware/kbd-nes-v2/nes_io.kicad_sch (KiCad schematic)
At the start: 13 parts, among them J1 Conn_01x05, J5 Conn_01x05, Q1 2N7002, SW1 SS12D07VG6 087

Commit message: Add key bindings reset - need to test - and also fix schematic and PCB for diode
Connections:
- net NES_5V_CLEAN: now also D1.1 (C); no longer D1.2 (A)
- net NES_IO_GND: now also D1.2 (A); no longer D1.1 (C)
Other:
- moved on the sheet: D1
Changed lines of the file:
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@@
 	(symbol
 		(lib_id "kbd-nes:SMAJ5.0A-13-F")
-		(at 149.86 127 90)
+		(at 149.86 127 270)
 		(unit 1)
 		(body_style 1)
@@
 		(fields_autoplaced yes)
 		(property "Reference" "D1"
-			(at 153.67 126.2399 90)
+			(at 153.67 125.2199 90)
 			(show_name no)
 			(do_not_autoplace no)
@@
 					(size 1.27 1.27)
 				)
-				(justify right)
+				(justify left)
 			)
 		)
 		(property "Value" "SMAJ5.0A-13-F"
-			(at 153.67 128.7799 90)
+			(at 153.67 127.7599 90)
 			(show_name no)
 			(do_not_autoplace no)
@@
 					(size 1.27 1.27)
 				)
-				(justify right)
+				(justify left)
 			)
 		)
 		(property "Footprint" "kbd-nes-pretty:SMA_L4.3-W2.6-LS5.2-RD"
-			(at 157.48 127 0)
+			(at 142.24 127 0)
 			(hide yes)
 			(show_name no)
@@
 		)
 		(property "Datasheet" "https://lcsc.com/product-detail/TVS_DIODES_SMAJ5-0A-13-F_SMAJ5-0A-13-F_C87074.html"
-			(at 160.02 127 0)
+			(at 139.7 127 0)
 			(hide yes)
 			(show_name no)
@@
 		)
 		(property "Manufacturer" "DIODES(美台)"
-			(at 162.56 127 0)
+			(at 137.16 127 0)
 			(hide yes)
 			(show_name no)
@@
 		)
 		(property "MPN" "SMAJ5.0A-13-F"
-			(at 165.1 127 0)
+			(at 134.62 127 0)
 			(hide yes)
 			(show_name no)
@@
 		)
 		(property "LCSC" "C87074"
-			(at 167.64 127 0)
+			(at 132.08 127 0)
 			(hide yes)
 			(show_name no)
